File: PCB/HerbUnitPCB/ESP32_S3.kicad_sch (KiCad schematic)
At the start: 28 parts, among them J1 USB_C_Receptacle_USB2.0_16P, J2 Barrel_Jack_Switch_Pin3Ring, SW1 SW_Push, SW2 SW_Push, U1 USBLC6-2P6, U2 ESP32-S3-WROOM-1, U3 AMS1117-5.0, U6 AP2112K-3.3

Commit message: Finished arrangement, fixed silkscreen
Parts:
- D5: footprint LED_SMD:LED_0201_0603Metric -> LED_SMD:LED_0402_1005Metric
Changed lines of the file:
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@@
 			)
 		)
-		(property "Footprint" "LED_SMD:LED_0201_0603Metric"
+		(property "Footprint" "LED_SMD:LED_0402_1005Metric"
 			(at 180.34 142.24 0)
 			(hide yes)

Commit message: PCB Routed + Silkscreen
Parts:
- added D6: Green LED, LED_SMD:LED_0402_1005Metric, symbol Device:LED
- added R16: 2k, Resistor_SMD:R_0402_1005Metric, symbol Device:R_US
Connections:
- net +3.3V_USB: now also R16.1
- net BlueLED: now also U2.29 (IO36); no longer U2.20 (IO12)
- net CalibrationButton: now also U2.22 (IO14); no longer U2.6 (IO6)
- net GND: now also D6.1 (K)
- net GreenLED: now also U2.30 (IO37); no longer U2.21 (IO13)
- net RedLED: now also U2.28 (IO35); no longer U2.19 (IO11)
- net TempSensor: now also U2.33 (IO40); no longer U2.5 (IO5)
- net WaterRead: now also U2.5 (IO5); no longer U2.18 (IO10)
- net VBUS: now reaches C3.1, D1.1 (K), J1.A4 (VBUS), J1.A9 (VBUS), J1.B4 (VBUS), J1.B9 (VBUS), R1.1
- net JACK_BUS: now reaches C5.1, J2.1, U3.3 (VI)
- new net: D6.2 (A), R16.2
Other:
- moved on the sheet: C6, C7, U6
