File: PCB/HerbUnitPCB/ESP32_S3.kicad_sch (KiCad schematic)
At the start: 30 parts, among them J1 USB_C_Receptacle_USB2.0_16P, J2 Barrel_Jack_Switch_Pin3Ring, SW1 SW_Push, SW2 SW_Push, U1 USBLC6-2P6, U2 ESP32-S3-WROOM-1, U3 AMS1117-5.0, U6 AP2112K-3.3

Commit message: Updated BOM to have all parts.
Parts:
- C1: MPN (none) -> GRM21BR61E226ME44K; Manufacturer (none) -> Murata Electronics
- C2, C8, C9: MPN (none) -> GRM155R62A104KE14D; Manufacturer (none) -> Murata Electronics
- C3, C4, C6, C7: footprint Capacitor_SMD:C_0805_2012Metric -> Capacitor_SMD:C_0402_1005Metric; MPN (none) -> GRM155R61A475MEAAD; Manufacturer (none) -> Murata Electronics
- C5: footprint Capacitor_SMD:C_0805_2012Metric -> Capacitor_SMD:C_1206_3216Metric; MPN (none) -> GRM319R61E106KA12D; Manufacturer (none) -> Murata Electronics
- D1: MPN (none) -> SOD882; Manufacturer (none) -> NXP
- D5, D6: footprint LED_SMD:LED_0402_1005Metric -> GreenLED:LED_APT2012CGCK
- J1: MPN (none) -> UJ31-CH-3-SMT-TR; Manufacturer (none) -> Same Sky
- J2: MPN (none) -> PJ-002A; Manufacturer (none) -> Same Sky
- R1: value 0 -> 330; MPN (none) -> RC0805FR-10330RL; Manufacturer (none) -> YAGEO
- R15, R16: MPN (none) -> AC0402FR-072KL; Manufacturer (none) -> YAGEO
- R2, R3, R5, R7: MPN (none) -> RT0402DRE075K1L; Manufacturer (none) -> YAGEO
- R4, R6, R8: MPN (none) -> RC0402FR-1310KL; Manufacturer (none) -> YAGEO
- SW1, SW2: value SW_Push -> BootButtons; MPN (none) -> B3U-1000P; Manufacturer (none) -> OMRON
- U1: MPN (none) -> USBLC6-2P6; Manufacturer (none) -> TECH PUBLIC
- U2: MPN (none) -> ESP32-S3-WROOM-1-N8; Manufacturer (none) -> ESPRESSIF
- U3: MPN (none) -> AMS1117-5.0(XBLW); Manufacturer (none) -> XBLW
- U6: MPN (none) -> AP2112K-3.3TRG1; Manufacturer (none) -> DIODES
