File: PCB/HerbUnitPCB/peripherals.kicad_sch (KiCad schematic)
At the start: 15 parts, among them J3 Conn_01x03_Pin, J4 SD_Card_Device, J5 Screw_Terminal_01x02, J6 Conn_01x03_Pin, SW3 SW_Push, U5 DHT11

Commit message: Finished arrangement, fixed silkscreen
Parts:
- SW3: footprint Button_Switch_SMD:SW_Push_1P1T_NO_CK_PTS125Sx43PSMTR -> Button_Switch_SMD:SW_Push_1P1T_NO_CK_PTS125Sx43SMTR
Changed lines of the file:
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@@
 			)
 		)
-		(property "Footprint" "Button_Switch_SMD:SW_Push_1P1T_NO_CK_PTS125Sx43PSMTR"
+		(property "Footprint" "Button_Switch_SMD:SW_Push_1P1T_NO_CK_PTS125Sx43SMTR"
 			(at 99.06 66.04 0)
 			(hide yes)

Commit message: PCB Routed + Silkscreen
Parts:
- J5: footprint TerminalBlock_Philmore:TerminalBlock_Philmore_TB132_1x02_P5.00mm_Horizontal -> TerminalBlock_Phoenix:TerminalBlock_Phoenix_MKDS-1,5-2-5.08_1x02_P5.08mm_Horizontal
Connections:
- net GreenLED: now also R10.1; no longer R13.1
- net RedLED: now also R13.1; no longer R10.1
Changed lines of the file:
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@@
+		)
+	)
+	(global_label "RedLED"
+		(shape input)
+		(at 29.21 59.69 180)
+		(fields_autoplaced yes)
+		(effects
+			(font
+				(size 1.27 1.27)
+			)
+			(justify right)
+		)
+		(property "Intersheetrefs" "${INTERSHEET_REFS}"
+			(at 19.2701 59.69 0)
+			(hide yes)
+			(show_name no)
+			(do_not_autoplace no)
+			(effects
+				(font
+					(size 1.27 1.27)
+				)
+				(justify right)
+			)
 		)
 	)
@@
 		)
 	)
-	(global_label "RedLED"
+	(global_label "GreenLED"
 		(shape input)
 		(at 29.21 33.02 180)
@@
 		)
 		(property "Intersheetrefs" "${INTERSHEET_REFS}"
-			(at 19.2701 33.02 0)
-			(hide yes)
-			(show_name no)
-			(do_not_autoplace no)
-			(effects
-				(font
-					(size 1.27 1.27)
-				)
-				(justify right)
-			)
-		)
-	)
-	(global_label "GreenLED"
-		(shape input)
-		(at 29.21 59.69 180)
-		(fields_autoplaced yes)
-		(effects
-			(font
-				(size 1.27 1.27)
-			)
-			(justify right)
-		)
-		(property "Intersheetrefs" "${INTERSHEET_REFS}"
-			(at 17.3953 59.69 0)
+			(at 17.3953 33.02 0)
 			(hide yes)
 			(show_name no)
@@
 			)
 		)
-		(property "Footprint" "TerminalBlock_Philmore:TerminalBlock_Philmore_TB132_1x02_P5.00mm_Horizontal"
+		(property "Footprint" "TerminalBlock_Phoenix:TerminalBlock_Phoenix_MKDS-1,5-2-5.08_1x02_P5.08mm_Horizontal"
 			(at 69.85 96.52 0)
 			(hide yes)
