File: PCB/HerbUnitPCB/peripherals.kicad_sch (KiCad schematic)
At the start: 15 parts, among them J3 Conn_01x03_Pin, J4 SD_Card_Device, J5 Screw_Terminal_01x02, J6 Conn_01x03_Pin, SW3 SW_Push, U5 DHT11

Commit message: Updated BOM to have all parts.
Parts:
- D2: MPN (none) -> APT2012CGCK; Manufacturer (none) -> Kingbright
- D3: MPN (none) -> APT2012VBC_D; Manufacturer (none) -> Kingbright
- D4: MPN (none) -> APT2012EC; Manufacturer (none) -> Kingbright
- J3, J6: MPN (none) -> 61300311021; Manufacturer (none) -> Würth Elektronik
- J4: MPN (none) -> MSD-3-A; Manufacturer (none) -> Same Sky
- J5: MPN (none) -> 1715721; Manufacturer (none) -> Phoenix Contact
- R10, R12, R13: MPN (none) -> AC0402FR-072KL; Manufacturer (none) -> YAGEO
- R11: MPN (none) -> RC0402FR-1310KL; Manufacturer (none) -> YAGEO
- R14: MPN (none) -> RT0805FRE0747KL; Manufacturer (none) -> YAGEO
- R9: MPN (none) -> RC0805JR-07100KL; Manufacturer (none) -> YAGEO
- SW3: value SW_Push -> CalibrationButton; MPN (none) -> PTS125SM43; Manufacturer (none) -> C&K
- U5: MPN (none) -> DHT11; Manufacturer (none) -> Aasong
