File: PCB/HerbUnitPCB/HerbUnitPCB.kicad_pcb (KiCad board)
At the start: 2 copper layers, 43 parts, among them J1 USB_C_Receptacle_USB2.0_16P, J2 Barrel_Jack_Switch_Pin3Ring, J3 Conn_01x03_Pin, J4 SD_Card_Device, J5 Screw_Terminal_01x02, J6 Conn_01x03_Pin, SW1 SW_Push, SW2 SW_Push, SW3 SW_Push, U1 USBLC6-2P6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

Commit message: PCB Routed + Silkscreen
Parts:
- added D6: Green LED, LED_SMD:LED_0402_1005Metric, F.Cu at (160.0, 89.5)
- added G***: LOGO, LOGO, F.Cu at (185.8, 61.3)
- added G***: LOGO, LOGO, B.Cu at (167.2, 44.6)
- added G***: LOGO, LOGO, B.Cu at (184.0, 89.6)
- added R16: 2k, Resistor_SMD:R_0402_1005Metric, F.Cu at (158.0, 86.7)
- C1, C2, R14, R9: moved to B.Cu
- J5: footprint TerminalBlock_Philmore:TerminalBlock_Philmore_TB132_1x02_P5.00mm_Horizontal -> TerminalBlock_Phoenix:TerminalBlock_Phoenix_MKDS-1,5-2-5.08_1x02_P5.08mm_Horizontal
- moved U6 27.4 mm to (157.3, 74.5), turned to 180 degrees
- moved C7 23.9 mm to (157.4, 77.4), turned to 0 degrees
- moved C6 22.6 mm to (160.5, 74.7), turned to 90 degrees
- moved C1 8.44 mm to (161.4, 36.8)
- moved D2 3.30 mm to (190.0, 86.4)
- moved D3 3.30 mm to (190.0, 90.2)
- moved D4 3.30 mm to (190.0, 94.0)
- moved R10 3.26 mm to (185.7, 86.4)
- moved C2 2.55 mm to (158.5, 36.7)
- moved R12 1.64 mm to (184.0, 90.2)
- moved SW3 1.30 mm to (167.4, 66.0)
- turned C4 to 180 degrees
Connections:
- net Net-(D1-K) renamed VBUS
- net Net-(U3-VI) renamed JACK_BUS
- R10 pad 1: RedLED -> GreenLED
- R13 pad 1: GreenLED -> RedLED
- U2 pad 18: WaterRead -> unconnected-(U2-IO10-Pad18)
- U2 pad 19: RedLED -> unconnected-(U2-IO11-Pad19)
- U2 pad 20: BlueLED -> unconnected-(U2-IO12-Pad20)
- U2 pad 21: GreenLED -> unconnected-(U2-IO13-Pad21)
- U2 pad 22: unconnected-(U2-IO14-Pad22) -> CalibrationButton
- U2 pad 28: unconnected-(U2-IO35-Pad28) -> RedLED
- U2 pad 29: unconnected-(U2-IO36-Pad29) -> BlueLED
- U2 pad 30: unconnected-(U2-IO37-Pad30) -> GreenLED
- U2 pad 33: unconnected-(U2-IO40-Pad33) -> TempSensor
- U2 pad 5: TempSensor -> WaterRead
- U2 pad 6: CalibrationButton -> unconnected-(U2-IO6-Pad6)
Routing:
- net +3.3V_USB: track 0.00 -> 165.5 mm, vias 0 -> 8
- net En: track 0.00 -> 54.7 mm, vias 0 -> 2
- net RedLED: track 0.00 -> 45.4 mm
- net BlueLED: track 0.00 -> 43.5 mm
- net GreenLED: track 0.00 -> 41.6 mm
- net BootMode1: track 0.00 -> 38.8 mm, vias 0 -> 2
- net SD_CS: track 0.00 -> 34.9 mm, vias 0 -> 2
- net USB_D-: track 0.00 -> 34.7 mm
- net USB_D+: track 0.00 -> 34.0 mm
- net SD_MOSI: track 0.00 -> 30.2 mm, vias 0 -> 2
- net CalibrationButton: track 0.00 -> 23.8 mm
- net MoistureRead: track 0.00 -> 22.4 mm
- net +5V_JACK: track 0.00 -> 20.4 mm
- net PumpMotor: track 0.00 -> 20.4 mm
- net TempSensor: track 0.00 -> 16.4 mm
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- added copper zone on B.Cu, net +3.3V_USB
- added copper zone on F.Cu, net +3.3V_USB
- added copper zone on F.Cu, net +5V
- added copper zone on B.Cu, net GND
- added copper zone on F.Cu, net GND
- added copper zone on In1.Cu, net GND
- added copper zone on In2.Cu, net GND
- added copper zone on F.Cu, net JACK_BUS
- added copper zone on F.Cu, net VBUS
Other:
- board outline added: 57.4 x 61.5 mm
- copper layers 2 -> 4
- board text added: "Boot"
- board text added: "Calibrate"
- board text added: "ESP PWR"
- board text added: "Float Sw."
- board text added: "Moist."
- board text added: "PUMP PWR"
- board text added: "Pump"
- board text added: "Pump PWR"
- board text added: "Reset"
- board text added: "SD Card Reader"
- board text added: "USB PWR"

Commit message: Started fabrication files
Parts:
- moved G*** 1.93 mm to (167.2, 46.5)
Changed lines of the file:
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@@
 		(capping no)
 		(filling no)
-		(zone_defaults)
 		(pcbplotparams
 			(layerselection 0x00000000_00000000_55555555_5755f5ff)
@@
 			(outputformat 1)
 			(mirror no)
-			(drillshape 1)
+			(drillshape 0)
 			(scaleselection 1)
-			(outputdirectory "")
+			(outputdirectory "Manufacturing/")
 		)
 	)
@@
 	(footprint "LOGO"
 		(layer "B.Cu")
-		(at 167.238 44.6024 180)
+		(at 167.238 46.5328 180)
 		(property "Reference" "G***"
 			(at 0 0 0)
@@
 	)
 	(segment
-		(start 158.488 39.902)
-		(end 152.3252 39.902)
-		(width 0.15)
+		(start 169.532 85.8644)
+		(end 169.5196 85.852)
+		(width 0.5)
 		(layer "F.Cu")
-		(net "MoistureRead")
+		(net "VBUS")
 	)
 	(segment
-		(start 150.1725 42.0547)
-		(end 150.1725 49.8875)
-		(width 0.15)
+		(start 169.532 87.122)
+		(end 169.532 85.8644)
+		(width 0.5)
 		(layer "F.Cu")
-		(net "MoistureRead")
+		(net "VBUS")
 	)
-	(segment
-		(start 152.3252 39.902)
-		(end 150.1725 42.0547)
-		(width 0.15)
-		(layer "F.Cu")
-		(net "MoistureRead")
+	(via
+		(at 164.6428 85.852)
+		(size 0.6)
+		(drill 0.3)
+		(layers "F.Cu" "B.Cu")
+		(net "VBUS")
 	)
-	(segment
-		(start 153.1535 52.8685)
-		(end 153.1535 54.055)
-		(width 0.15)
-		(layer "B.Cu")
-		(net "MoistureRead")
+	(via
+		(at 169.5196 85.852)
+		(size 0.6)
+		(drill 0.3)
+		(layers "F.Cu" "B.Cu")
+		(net "VBUS")
 	)
 	(segment
-		(start 150.1725 49.8875)
-		(end 153.1535 52.8685)
-		(width 0.15)
+		(start 169.5196 85.852)
+		(end 164.6428 85.852)
+		(width 0.5)
 		(layer "B.Cu")
-		(net "MoistureRead")
+		(net "VBUS")
 	)
 	(segment
@@
 	)
 	(segment
-		(start 169.532 85.8644)
-		(end 169.5196 85.852)
-		(width 0.5)
-		(layer "F.Cu")
-		(net "VBUS")
-	)
-	(segment
-		(start 169.532 87.122)
-		(end 169.532 85.8644)
-		(width 0.5)
-		(layer "F.Cu")
-		(net "VBUS")
-	)
-	(via
-		(at 164.6428 85.852)
-		(size 0.6)
-		(drill 0.3)
-		(layers "F.Cu" "B.Cu")
-		(net "VBUS")
-	)
-	(via
-		(at 169.5196 85.852)
-		(size 0.6)
-		(drill 0.3)
-		(layers "F.Cu" "B.Cu")
-		(net "VBUS")
-	)
-	(segment
-		(start 169.5196 85.852)
-		(end 164.6428 85.852)
-		(width 0.5)
-		(layer "B.Cu")
-		(net "VBUS")
-	)
-	(segment
 		(start 186.182 86.36)
 		(end 188.541 86.36)
@@
 	)
 	(segment
+		(start 158.4702 86.6648)
+		(end 158.4889 86.6648)
+		(width 0.15)
+		(layer "F.Cu")
+		(net "Net-(D6-A)")
+	)
+	(segment
+		(start 160.02 89.0595)
+		(end 160.02 88.2146)
+		(width 0.15)
+		(layer "F.Cu")
+		(net "Net-(D6-A)")
+	)
+	(segment
+		(start 160.02 88.2146)
+		(end 158.4702 86.6648)
+		(width 0.15)
+		(layer "F.Cu")
+		(net "Net-(D6-A)")
+	)
+	(segment
 		(start 160.4792 75.22379)
 		(end 160.4792 75.6494)
@@
 	)
 	(segment
+		(start 158.488 39.902)
+		(end 152.3252 39.902)
+		(width 0.15)
+		(layer "F.Cu")
+		(net "MoistureRead")
+	)
+	(segment
+		(start 150.1725 42.0547)
+		(end 150.1725 49.8875)
+		(width 0.15)
+		(layer "F.Cu")
+		(net "MoistureRead")
+	)
+	(segment
+		(start 152.3252 39.902)
+		(end 150.1725 42.0547)
+		(width 0.15)
+		(layer "F.Cu")
+		(net "MoistureRead")
+	)
+	(segment
+		(start 153.1535 52.8685)
+		(end 153.1535 54.055)
+		(width 0.15)
+		(layer "B.Cu")
+		(net "MoistureRead")
+	)
+	(segment
+		(start 150.1725 49.8875)
+		(end 153.1535 52.8685)
+		(width 0.15)
+		(layer "B.Cu")
+		(net "MoistureRead")
+	)
+	(segment
 		(start 180.34 79.502)
 		(end 180.34 80.518)
@@
 		(net "Net-(J5-Pin_2)")
 	)
-	(segment
-		(start 158.4702 86.6648)
-		(end 158.4889 86.6648)
-		(width 0.15)
-		(layer "F.Cu")
-		(net "Net-(D6-A)")
-	)
-	(segment
-		(start 160.02 89.0595)
-		(end 160.02 88.2146)
-		(width 0.15)
-		(layer "F.Cu")
-		(net "Net-(D6-A)")
-	)
-	(segment
-		(start 160.02 88.2146)
-		(end 158.4702 86.6648)
-		(width 0.15)
-		(layer "F.Cu")
-		(net "Net-(D6-A)")
-	)
 	(zone
